File: pcb/Delta_Robot.kicad_pcb (KiCad board)
At the start: 2 copper layers, 96.5 x 69.6 mm, 136 parts, among them IC1 STMPS2151MTR, J1 Conn_01x04, J2 Conn_01x03, J3 USB_A, J4 Conn_01x02, J5 Conn_01x02, J6 MP3V5050VC6U, J7 RJ45, J8 USB_OTG, J9 Conn_01x03, Q1 IRF9540STRLPBF, Q2 IRF9540STRLPBF, SW3 TL3305A, SW4 TL3305A, U2 LDL1117S33R, U3 ZLDO1117G12TA, U4 ICE40UP5K-SG48I, U5 W25Q64JVSSIQ, U6 STM32F412RGT6, U7 Omega2+, U8 4N25-X007T, U9 4N25-X007T, Y1 8MHz, Y2 32.768KHZ

Commit message: PCB finalizado (Enviado a fabricacion)
Parts:
- added C1: 0.1uF, Capacitor_SMD:C_0603_1608Metric, B.Cu at (139.1, 106.8)
- added R37: 100, Resistor_SMD:R_0603_1608Metric, F.Cu at (146.9, 88.9)
- added R38: 10k, Resistor_SMD:R_0603_1608Metric, F.Cu at (143.8, 88.9)
- moved R26 0.15 mm to (155.5, 109.8)
Connections:
- U7 pad 20: /FPGA/~FPGA_CRESET_B -> /FPGA/~FPGA_RESET
Routing:
- net +3V3: track 249.4 -> 259.2 mm
- net /Onion Omega 2/OMEGA2_JTAG_TMS: track 23.6 -> 28.3 mm
- net /Onion Omega 2/~OMEGA2_RST: track 11.8 -> 14.4 mm
- net /FPGA/~FPGA_RESET: track 0.00 -> 2.46 mm
- net /FPGA/~FPGA_CRESET_B: track 26.9 -> 24.8 mm
- net /Onion Omega 2/OMEGA2_JTAG_TDO: track 18.8 -> 20.9 mm
- net /FPGA/FPGA_SPI3: track 41.6 -> 43.2 mm
- net /Onion Omega 2/OMEGA2_JTAG_TCK: track 19.2 -> 20.8 mm
- net /Onion Omega 2/OMEGA2_JTAG_TRST: track 18.2 -> 19.7 mm
- net /STM32/STM32_USB_OverCurrent: track 16.7 -> 17.9 mm
- net /Onion Omega 2/OMEGA2_JTAG_TDI: track 18.6 -> 19.6 mm
- net /Onion Omega 2/Omega2_SER1_RX: track 16.3 -> 17.3 mm
- net /External Communications/EXT_I2C1: track 86.8 -> 87.6 mm
- net /FPGA/FPGA_SPI1: track 37.2 -> 37.9 mm, vias 2 -> 4
- net /Onion Omega 2/Omega2_SER1_TX: track 16.9 -> 17.5 mm
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Other:
- board text added: "24V"
- board text added: "5V"
- board text added: "DESIGNED BY: FRANCISCO PINTO 2020-5 v1.0"
- board text added: "GND"
- board text added: "GND PWR"
- board text added: "GND_PWR"
- board text added: "I2C_SCL"
- board text added: "I2C_SDA"
- board text added: "RS232_RX"
- board text added: "RS232_TX"
- board text added: "SOL1"
- board text added: "SOL2"
